File: Rosmo.kicad_pcb (KiCad board)
At the start: 2 copper layers, 88.4 x 99.3 mm, 107 parts, among them J1 C2904998, J2 C2904998, J3 C2904998, J4 C2904998, J5 CONN-SMD_4P-P1.00_SM04B-SRSS-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, P1 HDR-TH_2P-P2.54-V-F, P2 C2897365, U1 CONN-TH_DB125-2.54-10P-GN, U11 M3_STANDOFF, U12 M3_STANDOFF, U13 CONN-TH_DG308-2.54-02P-14-00A, U14 CONN-TH_DG308-2.54-02P-14-00A, U15 M3_STANDOFF, U16 HDR-TH_4P-P2.54-V-F, U17 M3_STANDOFF, U18 M3_STANDOFF, U19 M3_STANDOFF, U2 Pb, U20 N20-40MM-WHEEL, U21 N20-40MM-WHEEL, U22 RECTANGULAR_HOLE, U23 RECTANGULAR_HOLE, U24 N20-40MM-WHEEL, U25 M3_STANDOFF, U26 M3_STANDOFF, U29 RECTANGULAR_M3, U3 CONN-TH_DB125-2.54-10P-GN, U30 RECTANGULAR_M3, U31 RECTANGULAR_M3, U32 RECTANGULAR_M3, U33 CONN-TH_4P-P1.50_HCTL_HC-ZH1.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, U37 CONN-TH_DB125-2.54-10P-GN, U38 CONN-TH_DB125-2.54-10P-GN, U39 N20-40MM-WHEEL, U4 PWM, U40 RECTANGULAR_M3, U41 RECTANGULAR_M3, U42 RECTANGULAR_M3, U43 RECTANGULAR_M3, U45 C2895059, U46 CONN-TH_DG308-2.54-02P-14-00A, U48 C2895059, U49 C2895059, U5 HDR-TH_22P-P2.54-V-F, U50 HDR-TH_22P-P2.54-V-F, U51 HDR-TH_22P-P2.54-V-F, U6 C2895059, U7 HDR-TH_22P-P2.54-V-F, U8 RECTANGULAR_HOLE, U9 RECTANGULAR_HOLE

Commit message: update
Parts:
- removed H1A: C2905418, easyeda:HDR-TH_10P-P2.54-V-F
- removed H5: C50950, easyeda:HDR-TH_5P-P2.54-V-F
- removed P1: HDR-TH_2P-P2.54-V-F, easyeda:HDR-TH_2P-P2.54-V-F
- removed P2: C2897365, easyeda:HDR-TH_2P-P2.54-V-F
- removed U1, U37, U38: CONN-TH_DB125-2.54-10P-GN, easyeda:CONN-TH_DB125-2.54-10P-GN
- removed U4: PWM, easyeda:MIKROBUS_SILK
- removed U46: CONN-TH_DG308-2.54-02P-14-00A, easyeda:CONN-TH_DG308-2.54-02P-14-00A
- added P3: C2897365, easyeda:HDR-TH_2P-P2.54-V-F, F.Cu at (50.0, -19.9)
- added P4: HDR-TH_2P-P2.54-V-F, easyeda:HDR-TH_2P-P2.54-V-F, F.Cu at (60.3, -20.1)
- added QWIIC-LOGO-MEDIUM1: QWIIC-LOGO-MEDIUM, easyeda:QWIIC-LOGO-MEDIUM, F.Cu at (34.7, 29.0)
- added U28: CONN-TH_DB125-2.54-10P-GN, easyeda:CONN-TH_DB125-2.54-10P-GN, F.Cu at (38.2, 5.21)
- added U34: CONN-TH_DB125-2.54-10P-GN, easyeda:CONN-TH_DB125-2.54-10P-GN, F.Cu at (64.5, 5.21)
- added U52: CONN-TH_DB125-2.54-10P-GN, easyeda:CONN-TH_DB125-2.54-10P-GN, F.Cu at (38.0, 40.0)
- added U53: CONN-TH_DB125-2.54-10P-GN, easyeda:CONN-TH_DB125-2.54-10P-GN, F.Cu at (64.0, 40.0)
- added U55: PWM, easyeda:MIKROBUS_SILK, F.Cu at (54.4, -12.1)
- U16: value HDR-TH_4P-P2.54-V-F -> C2718488
- U3: value CONN-TH_DB125-2.54-10P-GN -> HDR-TH_6P-P2.54-H-F-W5.7; footprint easyeda:CONN-TH_DB125-2.54-10P-GN -> easyeda:HDR-TH_6P-P2.54-H-F-W5.7
- U33: value CONN-TH_4P-P1.50_HCTL_HC-ZH1.5-4AW -> C2845567
- U50, U51, U7: value HDR-TH_22P-P2.54-V-F -> C2886702
- moved U3 62.6 mm to (55.2, 65.5), turned to 0 degrees
- moved J5 7.19 mm to (40.4, 22.7)
- moved C12 5.85 mm to (45.6, 21.1), turned to 90 degrees
- moved U16 2.05 mm to (57.4, 47.6)
- moved .5 2.04 mm to (67.4, 56.1)
- moved C13 1.02 mm to (71.5, -20.2)
- moved ? 0.38 mm to (64.0, 64.8)
- moved R11 0.18 mm to (82.8, -20.6)
- moved U49 0.13 mm to (87.9, 58.9)
- moved U5 0.13 mm to (53.2, 35.6)
- moved U7 0.13 mm to (53.2, 13.1)
Connections:
- C1 pad 2: SER+ -> L1
- H6 pad 3: SER+ -> L1
- H6 pad 4: SER+ -> L1
- R11 pad 1: M2B -> M2CB
- R2 pad 1: M2A -> M2CA
- U3 pad 1: AN -> 3V
- U3 pad 2: RST -> GND
- U3 pad 3: E1B -> SCL
- U3 pad 4: CS -> SDA
- U3 pad 5: MOSI -> INT1
- U3 pad 6: CLK -> (no net)
- U5 pad 15: (no net) -> INT1
- U5 pad 16: (no net) -> SDA
- U5 pad 17: (no net) -> SCL
- U5 pad 18: (no net) -> 01
- U5 pad 2: (no net) -> E4B
- U5 pad 3: (no net) -> E4A
- U5 pad 4: (no net) -> M4CA
- U5 pad 5: (no net) -> M4CB
- U5 pad 6: (no net) -> SERB
- U5 pad 9: M1B -> M1CB
- U50 pad 10: (no net) -> AN
- U50 pad 11: (no net) -> 08
- U50 pad 12: (no net) -> RX
- U50 pad 13: (no net) -> TX
- U50 pad 14: (no net) -> M2CA
- U50 pad 15: (no net) -> M2CB
- U50 pad 16: (no net) -> E2A
- U50 pad 17: (no net) -> INT
- U50 pad 18: (no net) -> PWM
- U50 pad 19: (no net) -> E2B
- U50 pad 2: (no net) -> L1
- U50 pad 20: (no net) -> EN
- U50 pad 3: (no net) -> E1A
- U50 pad 4: (no net) -> MISO
- U50 pad 5: (no net) -> CLK
- U50 pad 6: (no net) -> CS
- U50 pad 7: (no net) -> MOSI
- U50 pad 8: (no net) -> E1B
- U50 pad 9: (no net) -> RST
- U51 pad 14: (no net) -> M1CB
- U51 pad 15: (no net) -> M3CB
- U51 pad 16: (no net) -> SERT
- U51 pad 18: (no net) -> M4CB
- U51 pad 19: (no net) -> M4CA
- U51 pad 20: (no net) -> E4A
- U51 pad 22: (no net) -> GND
- U51 pad 8: (no net) -> INT1
- U51 pad 9: (no net) -> M3A
- U6 pad 6: M2A -> M2CA
- U6 pad 7: M2B -> M2CB
- U7 pad 10: (no net) -> AN
- U7 pad 11: (no net) -> 08
- U7 pad 12: S$352450 -> RX
- U7 pad 13: S$352179 -> TX
- U7 pad 14: (no net) -> M2CA
- U7 pad 15: (no net) -> M2CB
- U7 pad 16: (no net) -> E2A
- U7 pad 17: (no net) -> INT
- U7 pad 18: (no net) -> PWM
- U7 pad 19: (no net) -> E2B
- U7 pad 20: (no net) -> EN
- U7 pad 22: (no net) -> 3V
- U7 pad 4: (no net) -> MISO
- U7 pad 5: (no net) -> CLK
- U7 pad 6: (no net) -> CS
- U7 pad 7: (no net) -> MOSI
- U7 pad 8: (no net) -> E1B
- U7 pad 9: (no net) -> RST
Routing:
- net GND: track 38.4 -> 473.8 mm, vias 17 -> 10
- net L1: track 71.1 -> 451.3 mm, vias 35 -> 23
- net M2CB: track 0.00 -> 67.2 mm, vias 0 -> 1
- net M2A: track 89.6 -> 26.1 mm, vias 2 -> 0
- net M2B: track 78.8 -> 17.0 mm
- net 3V: track 333.1 -> 275.9 mm, vias 8 -> 6
- net M2CA: track 0.00 -> 53.1 mm, vias 0 -> 1
- net M3CA: track 61.9 -> 8.89 mm, vias 4 -> 0
- net M3A: track 27.6 -> 56.8 mm, vias 0 -> 2
- net SCL: track 166.1 -> 137.4 mm, vias 3 -> 2
- net S$352179: track 23.5 -> 0.00 mm, vias 1 -> 0
- net S$352450: track 21.2 -> 0.00 mm, vias 1 -> 0
- net M1CB: track 101.7 -> 84.1 mm
- net M4CB: track 67.1 -> 56.2 mm
- net SDA: track 143.0 -> 133.4 mm, vias 5 -> 2
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Other:
- board text added: "01"
- board text added: "Brown"
- board text added: "CS"
- board text added: "Orange"
- board text added: "SerB"
- board text added: "SerTop"
- board text added: "x"
- board text removed: "BNO08x"
- board text removed: "CSO"
- board text removed: "Pi"
- board text removed: "Play"
- board text removed: "QWIIC"
- board text removed: "SC"
- board text removed: "SER"
- board text removed: "SERB"
- board text removed: "SERT"
- board text removed: "Zio Line follow"

Commit message: Added JLPCB production files
Parts:
- removed 20MM: ORP ORIGINAL 5X5 - NO EXTRA, easyeda:ORP ORIGINAL 5X5 - NO EXTRA
- removed the ? at (58.4, 21.3)
- removed the ? at (65.5, 48.3)
- removed the ? at (65.4, 2.79)
- removed the ? at (60.5, 21.3)
- removed the ? at (60.5, 23.2)
- removed the ? at (59.8, 51.9)
- removed the ? at (75.2, 56.0)
- removed C11, C13: C49678, easyeda:C0805
- removed R10: C17414, easyeda:R0805
- removed U29, U30, U31, U32, U40, U41, U42, U43: RECTANGULAR_M3, easyeda:RECTANGULAR_M3
- removed U55: PWM, easyeda:MIKROBUS_SILK
- added ?: , AutoGenerated:MountingHole_3.30mm, F.Cu at (65.7, 2.29)
- added ?: , AutoGenerated:MountingHole_3.30mm, F.Cu at (65.5, 48.1)
- added R1: C17414, easyeda:R0805, F.Cu at (89.2, 65.0)
- added U35: PWM, easyeda:MIKROBUS_SILK, F.Cu at (54.4, -12.1)
- added U38: ORP ROSMO - NO EXTRA, easyeda:ORP ROSMO - NO EXTRA, F.Cu at (65.7, 22.2)
- added U44: HOLECUT, easyeda:HOLECUT, F.Cu at (67.2, 68.8)
- added U46: HOLECUT, easyeda:HOLECUT, F.Cu at (42.2, 68.8)
- added U47: HOLECUT, easyeda:HOLECUT, F.Cu at (67.4, -25.3)
- added U54: HOLECUT, easyeda:HOLECUT, F.Cu at (41.3, -25.3)
- P4: value HDR-TH_2P-P2.54-V-F -> C49661
- U3: value HDR-TH_6P-P2.54-H-F-W5.7 -> C2833720
- moved C7 14.1 mm to (71.0, 28.8), turned to 180 degrees
- moved C6 10.8 mm to (70.2, 17.8), turned to 180 degrees
- moved R9 4.15 mm to (85.0, 65.2)
- moved C15 3.66 mm to (71.5, 51.7)
- moved U16 2.09 mm to (55.4, 48.1)
- moved C1 1.69 mm to (62.9, 24.0)
- moved .5 1.17 mm to (66.5, 55.4)
- moved U53 0.65 mm to (63.4, 39.9)
- moved U52 0.63 mm to (37.3, 40.0)
- moved U22 0.52 mm to (33.8, 55.1)
- moved U23 0.36 mm to (76.3, 55.1)
- moved U9 0.18 mm to (76.2, -20.6)
- moved C10 0.13 mm to (59.3, -15.2)
- moved U51 0.13 mm to (53.2, 35.6)
Connections:
- C5 pad 1: M4CB -> M4B
- C5 pad 2: M4CA -> M4A
- J1 pad 8: (no net) -> 3V
- J4 pad 1: M4CA -> M4A
- J4 pad 6: M4CB -> M4B
- U33 pad 1: S$352179 -> TX
- U33 pad 2: S$352450 -> RX
- U49 pad 1: M4CA -> M4A
- U49 pad 4: M4CB -> M4B
- U49 pad 7: M4CA -> MC4A
- U5 pad 14: M3A -> M3CA
- U5 pad 4: M4CA -> MC4A
- U51 pad 19: M4CA -> MC4A
- U51 pad 9: M3A -> M3CA
- U52 pad 2: M3A -> M3CA
- U53 pad 2: M4CA -> MC4A
Routing:
- net M4CA: track 75.6 -> 0.00 mm, vias 2 -> 0
- net MC4A: track 0.00 -> 55.6 mm
- net M3CA: track 8.89 -> 49.8 mm, vias 0 -> 1
- net RX: track 33.7 -> 69.7 mm
- net M4A: track 0.00 -> 27.2 mm
- net M3A: track 56.8 -> 31.8 mm
- net TX: track 30.1 -> 54.6 mm
- net M4B: track 0.00 -> 20.1 mm
- net E1B: track 29.6 -> 46.8 mm, vias 0 -> 1
- net SDA: track 133.4 -> 149.3 mm, vias 2 -> 1
- net SCL: track 137.4 -> 151.5 mm, vias 2 -> 1
- net M1CB: track 84.1 -> 97.4 mm, vias 1 -> 0
- net M4CB: track 56.2 -> 44.1 mm
- net M2CA: track 53.1 -> 63.8 mm
- net E4A: track 26.8 -> 17.1 mm
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Other:
- board size 88.4 x 99.3 mm -> 88 x 99.2 mm
- board text added: "SCK"
- board text added: "T"
- board text added: "Version 0.7"
- board text removed: "CLK"
- board text removed: "Version 0.5"
